File: Generator/illustration/schematic/schematic.kicad_sch (KiCad schematic)
At the start: 9 parts, among them U1 ESP32 devkit v1, U2 LCD 16bit 2 lines 16pins, U3 6v-24v dc to 5v dc, U4 Hall effect sensor, U5 ESC 3 phase motor

Commit message: working servo lib - just go broombroom and c the broombroom
Connections:
- net at U2. (VDD): now also RV2.2
- net at U1. (VP): now also U5. (VCC); no longer U2. (VDD)
- net at U5. (VCC): now also BT2.2 (-); no longer U1. (VP)
- new net: U1. (VP), U2. (VDD) (x6)
Changed lines of the file:
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@@
 (kicad_sch (version 20230121) (generator eeschema)
   (paper "A4")
+  (junction (at 100.33 60.96) (diameter 0) (color 0 0 0 0)
+  )
   (junction (at 163.83 48.26) (diameter 0) (color 0 0 0 0)
   )
@@
   (junction (at 171.45 49.53) (diameter 0) (color 0 0 0 0)
   )
+  (junction (at 111.76 63.5) (diameter 0) (color 0 0 0 0)
+  )
   (junction (at 101.6 60.96) (diameter 0) (color 0 0 0 0)
   )
@@
   (junction (at 111.76 120.65) (diameter 0) (color 0 0 0 0)
   )
-  (junction (at 100.33 60.96) (diameter 0) (color 0 0 0 0)
-  )
-  (junction (at 111.76 62.23) (diameter 0) (color 0 0 0 0)
-  )
   (junction (at 101.6 68.58) (diameter 0) (color 0 0 0 0)
   )
-  (wire (pts (xy 111.76 62.23) (xy 111.76 120.65))
-    (stroke (width 0) (type default))
-  )
   (wire (pts (xy 154.94 48.26) (xy 163.83 48.26))
     (stroke (width 0) (type default))
@@
     (stroke (width 0) (type default))
   )
-  (wire (pts (xy 58.42 62.23) (xy 111.76 62.23))
-    (stroke (width 0) (type default))
-  )
   (wire (pts (xy 55.88 118.11) (xy 55.88 130.81))
     (stroke (width 0) (type default))
@@
     (stroke (width 0) (type default))
   )
+  (wire (pts (xy 62.23 63.5) (xy 62.23 57.15))
+    (stroke (width 0) (type default))
+  )
   (wire (pts (xy 171.45 68.58) (xy 171.45 49.53))
     (stroke (width 0) (type default))
@@
     (stroke (width 0) (type default))
   )
-  (wire (pts (xy 62.23 57.15) (xy 62.23 60.96))
-    (stroke (width 0) (type default))
-  )
   (wire (pts (xy 73.66 72.39) (xy 73.66 57.15))
     (stroke (width 0) (type default))
@@
     (stroke (width 0) (type default))
   )
+  (wire (pts (xy 100.33 60.96) (xy 58.42 60.96))
+    (stroke (width 0) (type default))
+  )
+  (wire (pts (xy 111.76 63.5) (xy 111.76 120.65))
+    (stroke (width 0) (type default))
+  )
   (wire (pts (xy 133.35 31.75) (xy 151.13 31.75))
     (stroke (width 0) (type default))
@@
     (stroke (width 0) (type default))
   )
-  (wire (pts (xy 111.76 62.23) (xy 111.76 57.15))
+  (wire (pts (xy 111.76 57.15) (xy 111.76 63.5))
     (stroke (width 0) (type default))
   )
@@
     (stroke (width 0) (type default))
   )
-  (wire (pts (xy 100.33 60.96) (xy 62.23 60.96))
-    (stroke (width 0) (type default))
-  )
   (wire (pts (xy 82.55 88.9) (xy 82.55 72.39))
     (stroke (width 0) (type default))
@@
     (stroke (width 0) (type default))
   )
-  (wire (pts (xy 58.42 57.15) (xy 58.42 62.23))
-    (stroke (width 0) (type default))
-  )
   (wire (pts (xy 171.45 49.53) (xy 181.61 49.53))
     (stroke (width 0) (type default))
   )
+  (wire (pts (xy 111.76 63.5) (xy 62.23 63.5))
+    (stroke (width 0) (type default))
+  )
   (wire (pts (xy 71.12 82.55) (xy 104.14 82.55))
     (stroke (width 0) (type default))
@@
     (stroke (width 0) (type default))
   )
+  (wire (pts (xy 58.42 60.96) (xy 58.42 57.15))
+    (stroke (width 0) (type default))
+  )

Commit message: lezho
Parts:
- removed BT1: 11.1V Battery, symbol Device:Battery
- removed U3: 6v-24v dc to 5v dc, Module:Texas_EUS_R-PDSS-T5_THT, symbol Converter_DCDC:PTN78000H_EUS-5
- removed U5: ESC 3 phase motor, Package_DIP:DIP-8_W10.16mm, symbol esc:esc
- added M1: BLDC motor, symbol Motor:Motor_Servo
- added MES1: Ammeter_DC, symbol Device:Ammeter_DC
- added MES2: VOLTMETER_DC, symbol Device:Ammeter_DC
- added U3: ESP32 devkit v1, Package_SO:TSSOP-30_6.1x9.7mm_P0.65mm, symbol esp32-30pins:ESP32
- added U6: ESC 3 phase motor, Package_DIP:DIP-8_W10.16mm, symbol esc:esc
- BT2: value 7.4V Battery -> 11.1V Battery 30C
Connections:
- net at U4.2 (VOUT): now also U3. (VP); no longer U1. (VP)
- net at U2. (VDD): now also RV2.2
- net at U1. (VP): now also RV1.3; no longer U2. (VDD)
- net at BT2.1 (+): now also MES2.1 (-), U6. (VCC)
- net at BT2.2 (-): now also MES1.1 (-)
- new net: M1.1 (PWM), U6. (VCC)
- new net: M1.2 (+), U6. (VCC)
- new net: M1.3 (-), U6. (VCC)
- new net: U3. (VP), U4.1 (VCC)
- new net: U3. (VP), U4.3 (GND)
- new net: MES1.2 (+), MES2.2 (+), U6. (VCC)
- new net: RV2.1, U1. (VP), U2. (VDD), U6. (VCC)
- new net: RV2.3, U1. (VP), U2. (VDD), U6. (VCC)
- new net: U1. (VP), U2. (VDD) (x6)
- new net: U1. (VP), U6. (VCC)
Other:
- moved on the sheet: RV1, RV2
